File: Project_4_MCU_Datalogger/Project_4_MCU_Datalogger.kicad_sch (KiCad schematic)
At the start: 0 parts

Commit message: project 4 symbols added
Parts:
- added BT?: Battery, symbol Device:Battery
- added C1, C2, C3, C?: C, symbol Device:C
- added C?: C_Polarized, symbol Device:C_Polarized
- added D1, D?: LED, symbol Device:LED
- added H1, H2, H3, H?: MountingHole, symbol Mechanical:MountingHole
- added R1, R2, R3, R4, R5, R6, R?: R, symbol Device:R
- added U1, U?: 24LC1025, symbol Memory_EEPROM:24LC1025
- added U?: DS1337S_, DS1337S_:SOIC127P600X175-8N, symbol DS1337S_:DS1337S_
- added U?: ATMEGA328P-AU, ATMEGA328P-AU:QFP80P900X900X120-32N, symbol ATMEGA328P-AU:ATMEGA328P-AU
- added Y1, Y?: Crystal, symbol Device:Crystal
Connections:
- new net: U?.21 (GND), U?.3 (GND), U?.5 (GND)
- new net: U?.4 (VCC), U?.6 (VCC)
Other:
- added sheet Connectors (connectors.kicad_sch)

Commit message: project 4 symbols arranged
Parts:
- gave numbers to parts that had none: 10
- renumbered C1 to C2, C2 to C3, C3 to C4, D1 to D2, H1 to H2, H2 to H3, H3 to H4, R6 to R5, R5 to R6, U1 to U3, Y1 to Y2
Other:
- moved on the sheet: BT1, C1, C2, C3, C4, C5, D1, D2, H1, H2, H3, H4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

Commit message: project 4 added components values
Parts:
- C1, C4: value C -> 0.1u
- C2, C3: value C -> 22p
- C5: value C_Polarized -> 0.1u
- R1, R2, R6: value R -> 10K
- R3, R4: value R -> 4K7
- R5, R7: value R -> 330
- Y1: value Crystal -> 32.768 KHz
- Y2: value Crystal -> 16 MHz
Other:
- moved on the sheet: C4
Changed lines of the file:
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@@
 			)
 		)
-		(property "Value" "R"
+		(property "Value" "4K7"
 			(at 129.54 137.1599 0)
 			(effects
@@
 			)
 		)
-		(property "Value" "R"
+		(property "Value" "10K"
 			(at 104.14 44.4499 0)
 			(effects
@@
 			)
 		)
-		(property "Value" "Crystal"
+		(property "Value" "32.768 KHz"
 			(at 29.21 55.8799 90)
 			(effects
@@
 			)
 		)
-		(property "Value" "C_Polarized"
+		(property "Value" "0.1u"
 			(at 257.81 44.8309 0)
 			(effects
@@
 			)
 		)
-		(property "Value" "Crystal"
+		(property "Value" "16 MHz"
 			(at 171.45 71.12 0)
 			(effects
@@
 			)
 		)
-		(property "Value" "R"
+		(property "Value" "330"
 			(at 154.94 68.5799 0)
 			(effects
@@
 			)
 		)
-		(property "Value" "R"
+		(property "Value" "10K"
 			(at 116.84 44.4499 0)
 			(effects
@@
 			)
 		)
-		(property "Value" "C"
+		(property "Value" "0.1u"
 			(at 130.81 44.4499 0)
 			(effects
@@
 			)
 		)
-		(property "Value" "R"
+		(property "Value" "10K"
 			(at 198.12 93.9799 0)
 			(effects
@@
 			)
 		)
-		(property "Value" "R"
+		(property "Value" "330"
 			(at 243.84 55.8799 0)
 			(effects
@@
 			)
 		)
-		(property "Value" "R"
+		(property "Value" "4K7"
 			(at 116.84 137.1599 0)
 			(effects
@@
 	(symbol
 		(lib_id "Device:C")
-		(at 186.69 92.71 0)
+		(at 184.15 92.71 0)
 		(unit 1)
 		(exclude_from_sim no)
@@
 		(fields_autoplaced yes)
 		(property "Reference" "C4"
-			(at 190.5 91.4399 0)
-			(effects
-				(font
-					(size 1.27 1.27)
-				)
-				(justify left)
-			)
-		)
-		(property "Value" "C"
-			(at 190.5 93.9799 0)
+			(at 187.96 91.4399 0)
+			(effects
+				(font
+					(size 1.27 1.27)
+				)
+				(justify left)
+			)
+		)
+		(property "Value" "0.1u"
+			(at 187.96 93.9799 0)
 			(effects
 				(font
@@
 		)
 		(property "Footprint" ""
-			(at 187.6552 96.52 0)
+			(at 185.1152 96.52 0)
 			(effects
 				(font
@@
 		)
 		(property "Datasheet" "~"
-			(at 186.69 92.71 0)
+			(at 184.15 92.71 0)
 			(effects
 				(font
@@
 		)
 		(property "Description" "Unpolarized capacitor"
-			(at 186.69 92.71 0)
-			(effects
-				(font
-					(size 1.27 1.27)
-				)
-				(hide yes)
-			)
-		)
-		(property "Purpose" ""
-			(at 186.69 92.71 0)
+			(at 184.15 92.71 0)
+			(effects
+				(font
+					(size 1.27 1.27)
+				)
+				(hide yes)
+			)
+		)
+		(property "Purpose" ""
+			(at 184.15 92.71 0)
 			(effects
 				(font
@@
 			)
 		)
-		(property "Value" "C"
+		(property "Value" "22p"
 			(at 181.61 83.8199 0)
 			(effects
@@
 			)
 		)
-		(property "Value" "C"
+		(property "Value" "22p"
 			(at 168.91 83.8199 0)
 			(effects

Commit message: project 4 completed symbol-footprint associations
Parts:
- BT1: footprint (none) -> Connector_PinHeader_2.54mm:PinHeader_1x02_P2.54mm_Vertical
- C1, C2, C3, C4, C5: footprint (none) -> Capacitor_SMD:C_0805_2012Metric
- D1, D2: footprint (none) -> LED_SMD:LED_0805_2012Metric
- H1, H2, H3, H4: footprint (none) -> MountingHole:MountingHole_2.1mm
- R1, R2, R3, R4, R5, R6, R7: footprint (none) -> Resistor_SMD:R_0805_2012Metric
- U1, U3: footprint (none) -> Package_SO:SOIC-8_5.3x5.3mm_P1.27mm
- U2: footprint DS1337S_:SOIC127P600X175-8N -> Footprints:SOIC127P600X175-8N
- U4: footprint ATMEGA328P-AU:QFP80P900X900X120-32N -> Footprints:QFP80P900X900X120-32N
- Y1, Y2: footprint (none) -> Crystal:Crystal_SMD_5032-2Pin_5.0x3.2mm_HandSoldering
Other:
- moved on the sheet: C1, R1, R2, U2

Commit message: completed wiring
Connections:
- net VCC: now reaches R4.1
- net VCC: now also BT1.1 (+), C1.1, C5.1, D2.2 (A), R1.1, R2.1, R3.1, R6.1, U1.1 (A0), U1.2 (A1), U1.3 (A2), U1.8 (VCC), U2.8 (VCC), U3.1 (A0), U3.3 (A2), U3.8 (VCC), U4.18 (AVCC), U4.4 (VCC), U4.6 (VCC)
- net SDA: now reaches R4.2
- net SDA: now also U1.5 (SDA), U2.5 (SDA), U3.5 (SDA), U4.27 (PC4)
- net INTA: now reaches R1.2
- net INTA: now also U2.3 (~{INTA})
- net Y1_IN: now reaches U2.1 (X1)
- net Y1_IN: now also Y1.2
- net Y1_OUT: now reaches U2.2 (X2)
- net Y1_OUT: now also Y1.1
- net GND: now reaches U2.4 (GND)
- net GND: now also BT1.2 (-), C1.2, C2.2, C3.2, C4.2, C5.2, R5.2, R7.2, U1.4 (GND), U1.7 (WP), U3.2 (A1), U3.4 (GND), U3.7 (WP), U4.21 (GND), U4.3 (GND), U4.5 (GND)
- net SCL: now reaches U2.6 (SCL)
- net SCL: now also R3.2, U1.6 (SCL), U3.6 (SCL), U4.28 (PC5)
- net SQW: now reaches U2.7 (SQW/~INT)
- net SQW: now also R2.2
- net Y2_OUT: now reaches Y2.1
- net Y2_OUT: now also C3.1, U4.8 (PB7)
- net Y2_IN: now reaches Y2.2
- net Y2_IN: now also C2.1, U4.7 (PB6)
- net D1_K: now reaches R5.1
- net D1_K: now also D1.1 (K)
- net RESET: now reaches R6.2
- net RESET: now also U4.29 (PC6/~{RESET})
- net D3: now reaches U4.1 (PD3)
- net D6: now reaches U4.10 (PD6)
- net D7: now reaches U4.11 (PD7)
- net D8: now reaches U4.12 (PB0)
- net MOSI: now reaches U4.15 (PB3)
- net MISO: now reaches U4.16 (PB4)
- net SCLK: now reaches U4.17 (PB5)
- net SCLK: now also D1.2 (A)
- net D4: now reaches U4.2 (PD4)
- net AREF: now reaches U4.20 (AREF)
- net AREF: now also C4.1
- net RX: now reaches U4.30 (PD0)
- net TX: now reaches U4.31 (PD1)
- net D2: now reaches U4.32 (PD2)
- net D5: now reaches U4.9 (PD5)
- net D2_K: now reaches D2.1 (K)
- net D2_K: now also R7.1
- no-connect marks 0 -> 8
Other:
- sheet Connectors ports: added D2, D3, D4, D5, D6, D7, D8, GND, MISO, MOSI, RESET, RX, SCL, SCLK, SDA, TX, VCC; removed none
- note added: "Microcontrolador"
- note added: "Non-Volatile Memory"
- note added: "Real Time Clock"
- moved on the sheet: BT1, C1, C2, C3, C4, C5, D2, R1, R2, R3, R4, R5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

Commit message: schematic completed
Connections:
- net SCLK renamed SCK
- net Y1_IN renamed Y1_X1
- net Y1_OUT renamed Y1_X2
- net Y2_IN renamed XTAL_1
- net Y2_OUT renamed XTAL_2
Other:
- sheet Connectors ports: added SCK; removed SCLK
- note added: "EEPROM"
- note added: "MCU"
- note removed: "Microcontrolador"
- note removed: "Non-Volatile Memory"
- moved on the sheet: BT1, C2, C3, C4, C5, D2, R5, R6, R7, U4, Y2
